Commit message: Add existing project files to Git

File: interbotix_xsarm_descriptions/urdf/vx250.urdf.xacro (robot description, xacro)
@@ -17,14 +17,43 @@
     <texture filename="package://interbotix_xsarm_descriptions/meshes/interbotix_black.png"/>
   </material>
-  <xacro:if value="$(arg use_world_frame)">
-    <link name="world"/>
-    <joint name="fixed" type="fixed">
-      <parent link="world"/>
+  <material name="summit_black">
+    <texture filename="package://interbotix_xsarm_descriptions/meshes/summit_xl_gazebo.png"/>
+  </material>
+  <link name="Link0"/><!-- dummy -->
+  <joint name="dummy_joint" type="fixed">
+    <parent link="Link0"/>
+    <child link="base_box"/>
+      <origin xyz= "-0.05 0 0.185" rpy = " 0 0 0" />
+  </joint>
+  <link name="base_box">
+    <visual>
+      <origin rpy="0 0 ${pi/2}" xyz="-0.05 0 0"/>
+      <geometry>
+        <box size="0.3 0.3 0.37"/>
+      </geometry>
+      <material name="">
+        <color rgba="0.3 0.3 0.3 1"/>
+      </material>
+    </visual>
+    <collision>
+      <origin rpy="0 0 ${pi/2}" xyz="-0.05 0 0"/>
+      <geometry>
+        <box size="0.3 0.3 0.37"/>
+      </geometry>
+    </collision>
+    <inertial>
+      <origin rpy="0 0 ${pi/2}" xyz="0 0 0"/>
+      <mass value="100"/>
+      <inertia ixx="1.89" iyy="1.5" izz="1.89" ixy="0" ixz="0" iyz="0" />
+    </inertial>
+  </link>
+  <joint name="fixed" type="fixed">
+      <parent link="base_box"/>
       <child link="$(arg robot_name)/$(arg base_link_frame)"/>
-    </joint>
-  </xacro:if>
+        <origin xyz= "0 0 0" rpy = " 0 0 0" />
+  </joint>
   <link name="$(arg robot_name)/$(arg base_link_frame)">
     <visual>
-      <origin rpy="0 0 ${pi/2}" xyz="0 0 0"/>
+      <origin rpy="0 0 ${pi/2}" xyz="0 0 0.185"/>
       <geometry>
         <mesh filename="package://interbotix_xsarm_descriptions/meshes/vx250_meshes/vx250_1_base.stl" scale="0.001 0.001 0.001"/>
@@ -33,5 +62,5 @@
     </visual>
     <collision>
-      <origin rpy="0 0 ${pi/2}" xyz="0 0 0"/>
+      <origin rpy="0 0 ${pi/2}" xyz="0 0 0.185"/>
       <geometry>
         <mesh filename="package://interbotix_xsarm_descriptions/meshes/vx250_meshes/vx250_1_base.stl" scale="0.001 0.001 0.001"/>
@@ -63,5 +92,5 @@
   <link name="$(arg robot_name)/shoulder_link">
     <visual>
-      <origin rpy="0 0 ${pi/2}" xyz="0 0 -0.003"/>
+      <origin rpy="0 0 ${pi/2}" xyz="0 0 0.185"/>
       <geometry>
         <mesh filename="package://interbotix_xsarm_descriptions/meshes/vx250_meshes/vx250_2_shoulder.stl" scale="0.001 0.001 0.001"/>
@@ -70,5 +99,5 @@
     </visual>
     <collision>
-      <origin rpy="0 0 ${pi/2}" xyz="0 0 -0.003"/>
+      <origin rpy="0 0 ${pi/2}" xyz="0 0 0.185"/>
       <geometry>
         <mesh filename="package://interbotix_xsarm_descriptions/meshes/vx250_meshes/vx250_2_shoulder.stl" scale="0.001 0.001 0.001"/>
@@ -84,5 +113,5 @@
     <axis xyz="0 1 0"/>
     <limit effort="20" lower="${radians(-102)}" upper="${radians(100)}" velocity="${pi}"/>
-    <origin rpy="0 0 0" xyz="0 0 0.04805"/>
+    <origin rpy="0 0 0" xyz="0 0 0.23805"/>
     <parent link="$(arg robot_name)/shoulder_link"/>
     <child link="$(arg robot_name)/upper_arm_link"/>
